Commit message: new commit

File: robot_urdf_description/inertia.xacro (robot description, xacro)
@@ -5,27 +5,27 @@
 <xacro:macro name="inertia_of_sphere" params="mass radius *origin">
     <inertial>
-        <xacro:insert_block name ="origin"/>
+        <xacro:insert_block name="origin"/>
         <mass value="${mass}"/>
-        <inertia ixx="${(2/5)*mass*(radius*radius)}" ixy="0.0" ixz="0.0"
-                 iyy="${(2/5)*mass*(radius*radius)}"   iyz="0.0"
-                 izz="${(2/5)*mass*(radius*radius)}"/>
+        <inertia ixx="${(2.0/5.0) * mass * (radius * radius)}" ixy="0.0" ixz="0.0"
+                 iyy="${(2.0/5.0) * mass * (radius * radius)}" iyz="0.0"
+                 izz="${(2.0/5.0) * mass * (radius * radius)}"/>
     </inertial>
 </xacro:macro>
-<xacro:macro name="inertia_box" params="mass x y z *origin">
+<xacro:macro name="chassis_inertia" params="mass x y z *origin">
     <inertial>
-        <xacro:insert_block name ="origin"/>
+        <xacro:insert_block name="origin"/>
         <mass value="${mass}"/>
-        <inertia ixx="${(1/12)*mass*(y*y + z*z)}" ixy="0.0" ixz="0.0"
-                 iyy="${(1/12)*mass*(x*x + z*z)}"   iyz="0.0"
-                 izz="${(1/12)*mass*(x*x + y*y)}"/>
+        <inertia ixx="${(1.0/12.0) * mass * (y * y + z * z)}" ixy="0.0" ixz="0.0"
+                 iyy="${(1.0/12.0) * mass * (x * x + z * z)}" iyz="0.0"
+                 izz="${(1.0/12.0) * mass * (x * x + y * y)}"/>
     </inertial>
 </xacro:macro>
 <xacro:macro name="inertia_of_cylinder" params="mass length radius *origin">
     <inertial>
-        <xacro:insert_block name ="origin"/>
+        <xacro:insert_block name="origin"/>
         <mass value="${mass}"/>
-        <inertia ixx="${(1/12)*mass*(3*radius*radius + length*length)}" ixy="0.0" ixz="0.0"
-                 iyy="${(1/12)*mass*(3*radius*radius + length*length)}"   iyz="0.0"
-                 izz="${(1/12)*mass*(radius*radius)}"/>
+        <inertia ixx="${(1.0/12.0) * mass * (3 * radius * radius + length * length)}" ixy="0.0" ixz="0.0"
+                 iyy="${(1.0/12.0) * mass * (3 * radius * radius + length * length)}" iyz="0.0"
+                 izz="${(1.0/2.0) * mass * (radius * radius)}"/>
     </inertial>
 </xacro:macro>

File: robot_urdf_description/robot.urdf.xacro (robot description, xacro)
@@ -1,5 +1,9 @@
 <?xml version="1.0"?>
-<!-- http://wiki.ros.org/urdf/XML/link -->
-<robot xmlns:xacro="http://www.ros.org/wiki/xacro" name="my_robot">
-<xacro:include filename="urdf.xacro"/>
+<robot xmlns:xacro="http://www.ros.org/wiki/xacro" name="differential_robot">
+    <xacro:include filename="urdf.xacro"/>
+    <!--<xacro:include filename="gazebo.control.xacro"/>-->
+    <xacro:include filename="ros2Control.xacro"/>
+    <xacro:include filename="lidar.sensor.xacro"/>
+    <xacro:include filename="camera.xacro"/>
+    <!--<xacro:include filename="depth.camera.xacro"/>-->
 </robot>

File: robot_urdf_description/urdf.xacro (robot description, xacro)
@@ -1,121 +1,120 @@
 <?xml version="1.0"?>
-<!-- http://wiki.ros.org/urdf/XML/link -->
-<!-- using xacro for generating urdf file of the robot-->
 <robot xmlns:xacro="http://www.ros.org/wiki/xacro">
 <!--setting material properties which will be used later-->
 <xacro:include filename="inertia.xacro"/>
-<material name="white">
+<!-- Import the wheel macro -->
+<xacro:include filename="$(find my_robot)/robot_urdf_description/wheel_macro.xacro"/>
+<!-- Define properties -->
+<xacro:property name="x_dimension" value="0.3"/>
+<xacro:property name="y_dimension" value="0.3"/>
+<xacro:property name="z_dimension" value="0.15"/>
+<xacro:property name="wheel_length" value="0.04"/>
+<xacro:property name="wheel_radius" value="0.05"/>
+<xacro:property name="wheel_mass" value="0.1"/>
+<xacro:property name="chassis_mass" value="0.5"/>
+<!--constants-->
+<xacro:property name="PI" value="3.14159"/>
+<!-- setting material colors-->
+<material name="White">
     <color rgba="1 1 1 1"/>
 </material>
-<material name="orange">
+<material name="Orange">
     <color rgba="1 0.3 0.1 1"/>
 </material>
-<material name="blue">
+<material name="Blue">
     <color rgba="0.2 0.2 1 1"/>
 </material>
-<material name="black">
+<material name="Black">
     <color rgba="0 0 0 1"/>
+</material>
+<material name="Brown">
+    <color rgba="${222/255} ${207/255} ${195/255} 1.0"/>
+</material>
+<material name="Red">
+    <color rgba="0.96 0.26 0.21 1.0"/>
 </material>
 <!--setting up the base link-->
 <link name="base_link">
 </link>
-<!--joint name ="base_joint" type="fixed">
+<!-- adding base foot print link for simultanuous localization and mapping-->
+<link name="base_footprint">
+</link>
+<joint name ="base_footprint_joint" type="fixed">
     <parent link="base_link"/>
-    <child link="robot_chassis"/>
-</joint-->
-<!--setting up chassis link-->
-<link name="robot_chassis">
+    <child link="base_footprint"/>
+    <origin xyz="0 0 0" rpy="0 0 0"/>
+</joint>
+<!--################################# robot chassis link ###############################################-->
+<link name="chassis_link">
     <visual>
-        <origin xyz="0.15 0 0.075"/>
+        <origin xyz="${x_dimension/2} 0 ${z_dimension/2}"/> <!-- this is relative to chassis link-->
         <geometry>
-            <box size="0.3 0.3 0.15"/>
+            <box size="${x_dimension} ${y_dimension} ${z_dimension}"/>
         </geometry>
-        <material name= "white"/>
+        <material name="White"/>
     </visual>
     <collision>
-        <origin xyz="0.15 0 0.075"/>
+        <origin xyz="${x_dimension/2} 0 ${z_dimension/2}"/>
         <geometry>
-            <box size="0.3 0.3 0.15"/>
+            <box size="${x_dimension} ${y_dimension} ${z_dimension}"/>
         </geometry>
     </collision>
-    <xacro:inertia_box mass="0.5" x="0.3" y="0.3" z="0.15">
-        <origin xyz="0.15 0 0.075" rpy="0 0 0"/>
-    </xacro:inertia_box>
+    <xacro:chassis_inertia mass="${chassis_mass}" x="${x_dimension}" y="${y_dimension}" z="${z_dimension}">
+        <origin xyz="${x_dimension/2} 0 ${z_dimension/2}" rpy="0 0 0"/>
+    </xacro:chassis_inertia>
 </link>
 <joint name="chassis_joint" type="fixed">
     <parent link="base_link"/>
-    <child link="robot_chassis"/>
+    <child link="chassis_link"/>
     <origin xyz="-0.1 0 0"/>
 </joint>
-<!-- left wheel link-->
-<link name="left_wheel">
-    <visual>
-        <!--origin xyz="0.15 0 0.075" rpy="0 0 0"/-->
-        <geometry>
-            <cylinder radius="0.05" length= "0.04"/>
-        </geometry>
-        <material name= "blue"/>
-    </visual>
-    <collision>
-        <!--origin xyz="0.15 0 0.075"/-->
-        <geometry>
-            <cylinder radius="0.05" length= "0.04"/>
-        </geometry>
-    </collision>
-    <xacro:inertia_of_cylinder mass="0.1" radius="0.05" length= "0.04">
-        <origin xyz="0 0 0" rpy="0 0 0"/>
-    </xacro:inertia_of_cylinder>
-</link>
-<joint name="left_wheel_joint" type="continuous">
-    <parent link="base_link"/>
-    <child link="left_wheel"/>
-    <origin xyz="0 0.175 0" rpy="-${pi/2} 0 0"/>
-    <axis xyz="0 0 1"/>
-</joint>
-<!--right wheel link-->
-<link name="right_wheel">
-   <visual>
-        <geometry>
-            <cylinder radius="0.05" length="0.04"/>
-        </geometry>
-        <material name="blue"/>
-    </visual>
-    <collision>
-        <!--origin xyz="0.15 0 0.075"/-->
-        <geometry>
-            <cylinder radius="0.05" length= "0.04"/>
-        </geometry>
-    </collision>
-    <xacro:inertia_of_cylinder mass="0.1" radius="0.05" length= "0.04">
-        <origin xyz="0 0 0" rpy="0 0 0"/>
-    </xacro:inertia_of_cylinder>
-</link>
-<joint name="right_wheel_joint" type="continuous">
-    <parent link="base_link"/>
-    <child link="right_wheel"/>
-    <origin xyz="0 -0.175 0" rpy="${pi/2} 0 0"/>
-    <axis xyz="0 0 -1"/>
-</joint>
+<!-- adding gazebo reference for displaying the exact color of the robot-->
+<gazebo reference="chassis_link">
+    <material>Gazebo/White</material>
+</gazebo>
+<!--################################################################################################-->
+<!-- Use the macro for left and right wheels -->
+<xacro:wheel_link
+    wheel_name="left_wheel"
+    wheel_radius ="${wheel_radius}"
+    wheel_length ="${wheel_length}"
+    wheel_mass="${wheel_mass}"
+    y_offset="${y_dimension/2 + wheel_radius/2}"
+    axis_direction="-${PI/2}"
+    axis_of_rotation = "1" /> <!-- Indicates rotation of the wheels along the Z axis-->
+<xacro:wheel_link
+    wheel_name="right_wheel"
+    wheel_radius="${wheel_radius}"
+    wheel_length="${wheel_length}"
+    wheel_mass="${wheel_mass}"
+    y_offset="-${y_dimension/2 + wheel_radius/2}"
+    axis_direction="${PI/2}"
+    axis_of_rotation = "-1" /> <!-- Indicates rotation of the wheels along the Z axis-->
 <!-- caster wheel link-->
-<link name="caster_wheel">
+<link name="castor_wheel">
     <visual>
         <geometry>
-            <sphere radius="0.05"/>
+            <sphere radius="${wheel_radius}"/>
         </geometry>
-        <material name="black"/>
+        <material name="Black"/>
     </visual>
     <collision>
         <geometry>
-            <sphere radius="0.05"/>
+            <sphere radius="${wheel_radius}"/>
         </geometry>
     </collision>
-    <xacro:inertia_of_sphere mass="0.1" radius="0.05">
+    <xacro:inertia_of_sphere mass="${wheel_mass}" radius="${wheel_radius}">
         <origin xyz="0 0 0" rpy="0 0 0"/>
     </xacro:inertia_of_sphere>
 </link>
-<joint name="caster_wheel_joint" type="fixed">
-    <parent link="base_link"/>
-    <child link="caster_wheel"/>
-    <origin xyz="0.14 0 0"/>
+<gazebo reference="castor_wheel">
+    <material>Gazebo/Black</material>
+    <mu1 value="0.001"/>
+    <mu2 value="0.001"/>
+</gazebo>
+<joint name="castor_wheel_joint" type="fixed">
+    <parent link="chassis_link"/>
+    <child link="castor_wheel"/>
+    <origin xyz="0.24 0 0"/>
 </joint>
 </robot>
