Commit message: adding joystick control

File: robot_urdf_description/gazebo.control.xacro (robot description, xacro)
@@ -8,7 +8,7 @@
             <left_joint>left_wheel_joint</left_joint>
             <right_joint>right_wheel_joint</right_joint>
-            <!--wheel robot geometry-->
+            <!--wheel robot geometry /kinematics-->
             <wheel_separation>0.35</wheel_separation>
-            <wheel_radius>0.1</wheel_radius>
+            <wheel_radius>0.05</wheel_radius>
             <!-- limits-->
             <max_linear_acceleration>0.32</max_linear_acceleration>
@@ -17,6 +17,6 @@
             <!-- output-->
             <frame_id>odom</frame_id>
+            <odom_topic>odom</odom_topic>
             <child_frame_id>base_link</child_frame_id>
-            <odom_topic>odom</odom_topic>
             <odom_publisher_frequency>30</odom_publisher_frequency>
             <tf_topic>/tf</tf_topic>

File: robot_urdf_description/lidar.sensor.xacro (robot description, xacro)
@@ -6,4 +6,11 @@
         <geometry>
             <cylinder radius="0.05" length="0.04"/>
+        </geometry>
+        <material name="Orange"/>
+    </visual>
+    <visual>
+        <origin xyz="0 0 -0.05"/>
+        <geometry>
+            <cylinder radius ="0.01" length= "0.1"/>
         </geometry>
         <material name="Orange"/>
@@ -21,5 +28,5 @@
     <parent link="base_link"/>
     <child link="lidar_link"/>
-    <origin xyz="0.1 0 0.175" rpy="0 0 0"/>
+    <origin xyz="0.122 0 0.212" rpy="0 0 0"/>
     <axis xyz="0 0 0"/>
 </joint>
@@ -29,5 +36,5 @@
         <pose> 0 0 0 0 0 0 </pose>
         <visualize>true</visualize>
-        <!--<always_on>true</always_on>-->
+        <always_on>true</always_on>
         <update_rate>10</update_rate>
         <lidar>

File: robot_urdf_description/urdf.xacro (robot description, xacro)
@@ -45,5 +45,5 @@
     <origin xyz="0 0 0" rpy="0 0 0"/>
 </joint>
-<!--################################# robot chassis link ###############################################-->
+<!--##################### robot chassis link ##################-->
 <link name="chassis_link">
     <visual>
@@ -67,5 +67,5 @@
     <parent link="base_link"/>
     <child link="chassis_link"/>
-    <origin xyz="-0.1 0 0"/> <!-- this has be changed to wheel x and z offset after measurement-->
+    <origin xyz="-0.1 0 0"/> <!-- change to wheel x and z offset after measurement for real robot-->
 </joint>
  <!--adding gazebo reference for displaying the exact color of the robot-->
@@ -73,5 +73,5 @@
     <material>Gazebo/White</material>
 </gazebo>
-<!--################################################################################################-->
+<!--##*********************************************##-->
 <!-- Use the macro for left and right wheels -->
 <xacro:wheel_link

File: robot_urdf_description/wheel_macro.xacro (robot description, xacro)
@@ -21,4 +21,6 @@
         <gazebo reference="${wheel_name}">
             <material>Gazebo/Blue</material>
+            <mu1 value="0.5"/>
+            <mu2 value="0.5"/>
         </gazebo>
         <joint name="${wheel_name}_joint" type="continuous">
