Commit message: updating from gazebo classic to gazebo fortress

File: robot_urdf_description/camera.xacro (robot description, xacro)
@@ -1,9 +1,4 @@
 <?xml version="1.0"?>
 <robot xmlns:xacro="http://www.ros.org/wiki/xacro" >
-    <joint name="camera_joint" type="fixed">
-        <parent link="chassis_link"/>
-        <child link="camera_link"/>
-        <origin xyz="0.305 0 0.08" rpy="0 0 0"/>
-    </joint>
     <link name="camera_link">
         <visual>
@@ -14,4 +9,9 @@
         </visual>
     </link>
+    <joint name="camera_joint" type="fixed">
+        <parent link="chassis_link"/>
+        <child link="camera_link"/>
+        <origin xyz="0.305 0 0.08" rpy="0 0 0"/>
+    </joint>
     <joint name="camera_optical_joint" type="fixed">
         <parent link="camera_link"/>
@@ -21,7 +21,8 @@
     <link name="camera_link_optical"></link>
     <gazebo reference="camera_link">
-        <material>Gazebo/Red</material>
-        <sensor name="camera" type="camera">
+        <material name ="Red"/>
+        <sensor name="rgb_camera" type="camera">
             <pose> 0 0 0 0 0 0 </pose>
+            <always_on>true</always_on>
             <visualize>true</visualize>
             <update_rate>10</update_rate>
@@ -38,7 +39,6 @@
                 </clip>
             </camera>
-            <plugin name="camera_controller" filename="libgazebo_ros_camera.so">
-                <frame_name>camera_link_optical</frame_name>
-            </plugin>
+            <topic>camera/image_raw</topic>
+            <gz_frame_id>camera_link_optical</gz_frame_id> <!-- check out if camera works without this tag-->
         </sensor>
     </gazebo>

File: robot_urdf_description/gazebo.control.xacro (robot description, xacro)
@@ -4,19 +4,32 @@
     <gazebo>
     <!-- wheel information-->
-        <plugin name="diff_drive" filename="libgazebo_ros_diff_drive.so">
+        <plugin name="gz::sim::systems::DiffDrive" filename="gz-sim-diff-drive-system">
+            <!--wheel joints-->
             <left_joint>left_wheel_joint</left_joint>
             <right_joint>right_wheel_joint</right_joint>
+            <!--wheel robot geometry-->
             <wheel_separation>0.35</wheel_separation>
-            <wheel_diameter>0.1</wheel_diameter>
+            <wheel_radius>0.1</wheel_radius>
             <!-- limits-->
-            <max_wheel_torque>250</max_wheel_torque>
-            <max_wheel_acceleration>10.0</max_wheel_acceleration>
+            <max_linear_acceleration>0.32</max_linear_acceleration>
+            <!-- Input-->
+            <topic>cmd_vel</topic>
             <!-- output-->
-            <odometry_frame>odom</odometry_frame>
-            <robot_base_frame>base_link</robot_base_frame>
+            <frame_id>odom</frame_id>
+            <child_frame_id>base_link</child_frame_id>
+            <odom_topic>odom</odom_topic>
+            <odom_publisher_frequency>30</odom_publisher_frequency>
+            <tf_topic>/tf</tf_topic>
             <publish_odom>true</publish_odom>
             <publish_odom_tf>true</publish_odom_tf>
             <publish_wheel_tf>true</publish_wheel_tf>
         </plugin>
+        <!--== Joint state publisher ===-->
+        <plugin filename="gz-sim-joint-state-publisher-system"
+            name="gz::sim::systems::JointStatePublisher">
+            <topic>joint_states</topic>
+            <joint_name>left_wheel_joint</joint_name>
+            <joint_name>right_wheel_joint</joint_name>
+        </plugin>
     </gazebo>
 </robot>

File: robot_urdf_description/lidar.sensor.xacro (robot description, xacro)
@@ -2,5 +2,5 @@
 <!-- http://wiki.ros.org/urdf/XML/link -->
 <robot xmlns:xacro="http://www.ros.org/wiki/xacro">
-<link name="lidar_sensor">
+<link name="lidar_link">
    <visual>
         <geometry>
@@ -10,5 +10,4 @@
     </visual>
     <collision>
-        <!--origin xyz="0.15 0 0.075"/-->
         <geometry>
             <cylinder radius="0.05" length= "0.04"/>
@@ -19,11 +18,18 @@
     </xacro:inertia_of_cylinder>
 </link>
-<gazebo reference="lidar_sensor">
-    <material>Gazebo/Orange</material>
-    <sensor name="laser" type="ray">
+<joint name="lidar_link_joint" type="fixed">
+    <parent link="base_link"/>
+    <child link="lidar_link"/>
+    <origin xyz="0.1 0 0.175" rpy="0 0 0"/>
+    <axis xyz="0 0 0"/>
+</joint>
+<gazebo reference="lidar_link"> <!--changed lidar_link to lidar_link-->
+    <material name="Orange"/>
+    <sensor name="lidar_link" type="gpu_lidar">
         <pose> 0 0 0 0 0 0 </pose>
-        <visualize>false</visualize>
+        <visualize>true</visualize>
+        <!--<always_on>true</always_on>-->
         <update_rate>10</update_rate>
-        <ray>
+        <lidar>
             <scan>
                 <horizontal>
@@ -37,19 +43,8 @@
                     <max>12</max>
                 </range>
-        </ray>
-        <plugin name="laser_controller" filename="libgazebo_ros_ray_sensor.so">
-                <ros>
-                    <argument>~/out:=scan</argument>
-                </ros>
-                <output_type>sensor_msgs/LaserScan</output_type>
-                <frame_name>lidar_sensor</frame_name>
-        </plugin>
+        </lidar>
+        <gz_frame_id>lidar_link</gz_frame_id>
+        <topic>scan</topic>
     </sensor>
 </gazebo>
-<joint name="lidar_sensor_joint" type="fixed">
-    <parent link="base_link"/>
-    <child link="lidar_sensor"/>
-    <origin xyz="0.1 0 0.175" rpy="0 0 0"/>
-    <axis xyz="0 0 0"/>
-</joint>
 </robot>

File: robot_urdf_description/ros2Control.xacro (robot description, xacro)
@@ -4,5 +4,5 @@
     <ros2_control name="GazeboSystem" type="system">
         <hardware>
-            <plugin>gazebo_ros2_control/GazeboSystem</plugin>
+            <plugin>gz_ros2_control/GazeboSimSystem</plugin>
         </hardware>
         <joint name="left_wheel_joint">
@@ -24,5 +24,6 @@
     </ros2_control>
     <gazebo>
-        <plugin name="gazebo_ros2_control" filename="libgazebo_ros2_control.so">
+        <plugin name="gz_ros2_control::GazeboSimROS2ControlPlugin"
+            filename="libgz_ros2_control-system.so">
             <parameters>$(find my_robot)/config/controller.yaml</parameters>
         </plugin>

File: robot_urdf_description/urdf.xacro (robot description, xacro)
@@ -67,7 +67,7 @@
     <parent link="base_link"/>
     <child link="chassis_link"/>
-    <origin xyz="-0.1 0 0"/>
+    <origin xyz="-0.1 0 0"/> <!-- this has be changed to wheel x and z offset after measurement-->
 </joint>
-<!-- adding gazebo reference for displaying the exact color of the robot-->
+ <!--adding gazebo reference for displaying the exact color of the robot-->
 <gazebo reference="chassis_link">
     <material>Gazebo/White</material>

Commit message: Update URDF to match the physical robot

File: robot_urdf_description/camera.xacro (robot description, xacro)
@@ -6,5 +6,5 @@
                 <box size="0.010 0.03 0.03"/>
             </geometry>
-            <material name="Red"/>
+            <material name="Blue"/>
         </visual>
     </link>
@@ -12,5 +12,5 @@
         <parent link="chassis_link"/>
         <child link="camera_link"/>
-        <origin xyz="0.305 0 0.08" rpy="0 0 0"/>
+        <origin xyz="0.255 0 0.1" rpy="0 0 0"/>
     </joint>
     <joint name="camera_optical_joint" type="fixed">
@@ -21,9 +21,9 @@
     <link name="camera_link_optical"></link>
     <gazebo reference="camera_link">
-        <material name ="Red"/>
+        <material name ="Blue"/>
         <sensor name="rgb_camera" type="camera">
             <pose> 0 0 0 0 0 0 </pose>
             <always_on>true</always_on>
-            <visualize>true</visualize>
+            <visualize>false</visualize>
             <update_rate>10</update_rate>
             <camera>

File: robot_urdf_description/gazebo.control.xacro (robot description, xacro)
@@ -9,6 +9,6 @@
             <right_joint>right_wheel_joint</right_joint>
             <!--wheel robot geometry /kinematics-->
-            <wheel_separation>0.35</wheel_separation>
-            <wheel_radius>0.05</wheel_radius>
+            <wheel_separation>0.195</wheel_separation>
+            <wheel_radius>0.0325</wheel_radius>
             <!-- limits-->
             <max_linear_acceleration>0.32</max_linear_acceleration>

File: robot_urdf_description/lidar.sensor.xacro (robot description, xacro)
@@ -2,24 +2,33 @@
 <!-- http://wiki.ros.org/urdf/XML/link -->
 <robot xmlns:xacro="http://www.ros.org/wiki/xacro">
+<!-- Dimensions for the LiDAR sensor-->
+<xacro:property name="lidar_offset_x" value="0.16"/> <!-- relative to base link-->
+<xacro:property name="lidar_offset_chassis_z" value="0.18"/> <!-- relative to chassis-->
+<xacro:property name="lidar_offset_z" value="${lidar_offset_chassis_z + chassis_offset_z}"/> <!-- relative to base link-->
+<xacro:property name= "lidar_radius" value="0.0345"/>
+<xacro:property name= "lidar_height" value="0.023"/>
+<xacro:property name= "lidar_spacer_height" value="0.1"/>
+<xacro:property name= "lidar_spacer_radius" value= "0.01"/>
 <link name="lidar_link">
    <visual>
         <geometry>
-            <cylinder radius="0.05" length="0.04"/>
+            <cylinder radius="${lidar_radius}" length="${lidar_height}"/>
         </geometry>
-        <material name="Orange"/>
+        <material name="Dark"/>
     </visual>
+<!-- visual for LiDAR spacer -->
     <visual>
-        <origin xyz="0 0 -0.05"/>
+        <origin xyz="0 0 -${lidar_height/2 + lidar_spacer_height/2}"/>
         <geometry>
-            <cylinder radius ="0.01" length= "0.1"/>
+            <cylinder radius ="${lidar_spacer_radius}" length= "${lidar_spacer_height}"/>
         </geometry>
-        <material name="Orange"/>
+        <material name="Dark"/>
     </visual>
     <collision>
         <geometry>
-            <cylinder radius="0.05" length= "0.04"/>
+            <cylinder radius="${lidar_radius}" length="${lidar_height}"/>
         </geometry>
     </collision>
-    <xacro:inertia_of_cylinder mass="0.1" radius="0.05" length= "0.04">
+    <xacro:inertia_of_cylinder mass="0.06" radius="${lidar_radius}" length="${lidar_height}">
         <origin xyz="0 0 0" rpy="0 0 0"/>
     </xacro:inertia_of_cylinder>
@@ -28,9 +37,9 @@
     <parent link="base_link"/>
     <child link="lidar_link"/>
-    <origin xyz="0.122 0 0.212" rpy="0 0 0"/>
+    <origin xyz="${lidar_offset_x} 0 ${lidar_offset_z}" rpy="0 0 0"/>
     <axis xyz="0 0 0"/>
 </joint>
 <gazebo reference="lidar_link"> <!--changed lidar_link to lidar_link-->
-    <material name="Orange"/>
+    <material name="Dark"/>
     <sensor name="lidar_link" type="gpu_lidar">
         <pose> 0 0 0 0 0 0 </pose>
@@ -41,5 +50,5 @@
             <scan>
                 <horizontal>
-                    <samples>360</samples>
+                    <samples>90</samples>
                     <min_angle>-3.14</min_angle>
                     <max_angle>3.14</max_angle>

File: robot_urdf_description/robot.urdf.xacro (robot description, xacro)
@@ -2,5 +2,5 @@
 <robot xmlns:xacro="http://www.ros.org/wiki/xacro" name="differential_robot">
     <xacro:include filename="urdf.xacro"/>
-    <!--<xacro:include filename="gazebo.control.xacro"/>-->
+    <xacro:include filename="gazebo.control.xacro"/>
     <xacro:include filename="ros2Control.xacro"/>
     <xacro:include filename="lidar.sensor.xacro"/>

File: robot_urdf_description/urdf.xacro (robot description, xacro)
@@ -5,12 +5,23 @@
 <!-- Import the wheel macro -->
 <xacro:include filename="$(find my_robot)/robot_urdf_description/wheel_macro.xacro"/>
-<!-- Define properties -->
-<xacro:property name="x_dimension" value="0.3"/>
-<xacro:property name="y_dimension" value="0.3"/>
-<xacro:property name="z_dimension" value="0.15"/>
-<xacro:property name="wheel_length" value="0.04"/>
-<xacro:property name="wheel_radius" value="0.05"/>
-<xacro:property name="wheel_mass" value="0.1"/>
-<xacro:property name="chassis_mass" value="0.5"/>
+<!-- Define chassisproperties -->
+<xacro:property name="chassis_length" value="0.25"/>
+<xacro:property name="chassis_width" value="0.17"/>
+<xacro:property name="chassis_height" value="0.14"/>
+<xacro:property name="chassis_mass" value="0.7"/>
+<xacro:property name="chassis_offset_x" value="0.045"/> <!-- relative base link-->
+<xacro:property name= "chassis_offset_z" value= "0.023"/> <!-- relative base link-->
+<!--  wheel properties -->
+<xacro:property name="driven_wheel_thickness" value="0.026"/>
+<xacro:property name="driven_wheel_radius" value="0.0325"/>
+<xacro:property name="driven_wheel_mass" value="0.02"/> <!--change with actual mass -->
+<xacro:property name="driven_wheel_offset_y" value ="0.0975"/> <!-- relative to base link-->
+<!--  castor wheel properties -->
+<xacro:property name="castor_wheel_thickness" value="0.022"/> <!--used for cylinderical castor wheel-->
+<xacro:property name="castor_wheel_radius" value="0.019"/>
+<xacro:property name="castor_wheel_mass" value="0.01"/> <!--change with actual mass -->
+<xacro:property name= "castor_wheel_offset_x" value="0.215"/>
+<!--<xacro:property name= "castor_wheel_offset_z" value="${-driven_wheel_radius + castor_wheel_radius}"/> --><!-- relative to chassis-->
+<xacro:property name= "castor_wheel_offset_z" value="${-0.036}"/> <!-- relative to chassis-->
 <!--constants-->
 <xacro:property name="PI" value="3.14159"/>
@@ -34,4 +45,16 @@
     <color rgba="0.96 0.26 0.21 1.0"/>
 </material>
+<material name="Dark">
+    <color rgba="0.3 0.3 0.3 1.0"/>
+</material>
+<material name="light_black">
+    <color rgba="0.4 0.4 0.4 1.0"/>
+</material>
+<material name="green">
+    <color rgba="0.0 0.8 0.0 1.0"/>
+  </material>
+  <material name="grey">
+    <color rgba="0.5 0.5 0.5 1.0"/>
+  </material>
 <!--setting up the base link-->
 <link name="base_link">
@@ -48,18 +71,18 @@
 <link name="chassis_link">
     <visual>
-        <origin xyz="${x_dimension/2} 0 ${z_dimension/2}"/> <!-- this is relative to chassis link-->
+        <origin xyz="${chassis_length/2} 0 ${chassis_height/2}"/> <!-- this is relative to chassis link-->
         <geometry>
-            <box size="${x_dimension} ${y_dimension} ${z_dimension}"/>
+            <box size="${chassis_length} ${chassis_width} ${chassis_height}"/>
         </geometry>
-        <material name="White"/>
+        <material name="Red"/>
     </visual>
     <collision>
-        <origin xyz="${x_dimension/2} 0 ${z_dimension/2}"/>
+        <origin xyz="${chassis_length/2} 0 ${chassis_height/2}"/>
         <geometry>
-            <box size="${x_dimension} ${y_dimension} ${z_dimension}"/>
+            <box size="${chassis_length} ${chassis_width} ${chassis_height}"/>
         </geometry>
     </collision>
-    <xacro:chassis_inertia mass="${chassis_mass}" x="${x_dimension}" y="${y_dimension}" z="${z_dimension}">
-        <origin xyz="${x_dimension/2} 0 ${z_dimension/2}" rpy="0 0 0"/>
+    <xacro:chassis_inertia mass="${chassis_mass}" x="${chassis_length}" y="${chassis_width}" z="${chassis_height}">
+        <origin xyz="${chassis_length/2} 0 ${chassis_height/2}" rpy="0 0 0"/>
     </xacro:chassis_inertia>
 </link>
@@ -67,9 +90,9 @@
     <parent link="base_link"/>
     <child link="chassis_link"/>
-    <origin xyz="-0.1 0 0"/> <!-- change to wheel x and z offset after measurement for real robot-->
+    <origin xyz="${-chassis_offset_x} 0 ${chassis_offset_z}"/> <!-- change to wheel x and z offset after measurement for real robot-->
 </joint>
  <!--adding gazebo reference for displaying the exact color of the robot-->
 <gazebo reference="chassis_link">
-    <material>Gazebo/White</material>
+    <material>Gazebo/Red</material>
 </gazebo>
 <!--##*********************************************##-->
@@ -77,16 +100,16 @@
 <xacro:wheel_link
     wheel_name="left_wheel"
-    wheel_radius ="${wheel_radius}"
-    wheel_length ="${wheel_length}"
-    wheel_mass="${wheel_mass}"
-    y_offset="${y_dimension/2 + wheel_radius/2}"
+    wheel_radius ="${driven_wheel_radius}"
+    wheel_length ="${driven_wheel_thickness}"
+    wheel_mass="${driven_wheel_mass}"
+    y_offset="${driven_wheel_offset_y}"
     axis_direction="-${PI/2}"
     axis_of_rotation = "1" /> <!-- Indicates rotation of the wheels along the Z axis-->
 <xacro:wheel_link
     wheel_name="right_wheel"
-    wheel_radius="${wheel_radius}"
-    wheel_length="${wheel_length}"
-    wheel_mass="${wheel_mass}"
-    y_offset="-${y_dimension/2 + wheel_radius/2}"
+    wheel_radius="${driven_wheel_radius}"
+    wheel_length="${driven_wheel_thickness}"
+    wheel_mass="${driven_wheel_mass}"
+    y_offset="-${driven_wheel_offset_y}"
     axis_direction="${PI/2}"
     axis_of_rotation = "-1" /> <!-- Indicates rotation of the wheels along the Z axis-->
@@ -95,5 +118,5 @@
     <visual>
         <geometry>
-            <sphere radius="${wheel_radius}"/>
+            <sphere radius="${castor_wheel_radius}"/>
         </geometry>
         <material name="Black"/>
@@ -101,8 +124,8 @@
     <collision>
         <geometry>
-            <sphere radius="${wheel_radius}"/>
+            <sphere radius="${castor_wheel_radius}"/>
         </geometry>
     </collision>
-    <xacro:inertia_of_sphere mass="${wheel_mass}" radius="${wheel_radius}">
+    <xacro:inertia_of_sphere mass="${castor_wheel_mass}" radius="${castor_wheel_radius}">
         <origin xyz="0 0 0" rpy="0 0 0"/>
     </xacro:inertia_of_sphere>
@@ -116,5 +139,5 @@
     <parent link="chassis_link"/>
     <child link="castor_wheel"/>
-    <origin xyz="0.24 0 0"/>
+    <origin xyz="${castor_wheel_offset_x} 0 ${castor_wheel_offset_z}"/>
 </joint>
 </robot>
